Commit message: adding all code since it's deciding to play up

File: data/laikago/laikago.urdf (robot description, URDF)
Before this commit: robot plane, 13 links, 12 joints
Links:
- link FR_hip_motor: mass 0.241 -> 1.095
- link RR_hip_motor: mass 0.241 -> 1.095

File: data/laikago_long_legs/laikago.urdf (robot description, URDF)
Before this commit: robot plane, 13 links, 12 joints
Links:
- link FR_hip_motor: mass 0.241 -> 1.095
