Commit message: Adding experiments, as well as sh script

File: data/laikago_long_legs/laikago.urdf (robot description, URDF)
Before this commit: robot plane, 13 links, 12 joints
Links:
- link FL_lower_leg: geometry collision mesh filename=lower_leg_3.stl scale=1 1.5 1; visual mesh filename=lower_leg_3.stl scale=1 1.5 1
- link FR_lower_leg: geometry collision mesh filename=lower_leg_3.stl scale=1 1.5 1; visual mesh filename=lower_leg_3.stl scale=1 1.5 1
- link RL_lower_leg: geometry collision mesh filename=lower_leg_3.stl scale=1 1.5 1; visual mesh filename=lower_leg_3.stl scale=1 1.5 1
- link RR_hip_motor: mass 0.241 -> 1.095
- link RR_lower_leg: geometry collision mesh filename=lower_leg_3.stl scale=1 1.5 1; visual mesh filename=lower_leg_3.stl scale=1 1.5 1
- link chassis: mass 20 -> 13.715
